File: pcb/photodiode.sch (KiCad schematic (older format))
At the start: 9 parts, among them U6 photodiode, U7 LM324N

Commit message: fix µcu farnell code
Connections:
- net DIO: now also U7.14; no longer U7.7
- net at C11.2, R13.1: now also U7.12 (+); no longer U7.5 (+)
- net at U6.2 (C): now also U7.9 (-); no longer U7.2 (-)
- net at R11.1: now also U7.10 (+); no longer U7.3 (+)
- net at R11.2, R12.2: now also U7.8; no longer U7.1
- net at R14.1, R15.2: now also U7.13 (-); no longer U7.6 (-)
Changed lines of the file:
@@
 AR Path="/55BDA313/55BD9EC1" Ref="U5"  Part="1"
 AR Path="/55BDA511/55BD9EC1" Ref="U8"  Part="1"
-F 0 "U3" H 3350 3600 60  0000 C CNN
+F 0 "U8" H 3350 3600 60  0000 C CNN
 F 1 "photodiode" H 3350 3600 60  0000 C CNN
 F 2 "" H 3350 3600 60  0000 C CNN
@@
 AR Path="/55BDA313/55BD9EC8" Ref="R6"  Part="1"
 AR Path="/55BDA511/55BD9EC8" Ref="R16"  Part="1"
-F 0 "R1" V 4425 2750 50  0000 C CNN
+F 0 "R16" V 4425 2750 50  0000 C CNN
 F 1 "UNREGULATED" V 4525 2775 50  0000 C CNN
 F 2 "" V 4330 2750 30  0000 C CNN
@@
 $EndComp
 $Comp
-L GNDA #PWR021
+L GNDA #PWR39
 U 1 1 55BD9ECF
 P 3475 3925
-AR Path="/55BDA44F/55BD9ECF" Ref="#PWR021"  Part="1"
-AR Path="/55BD9D56/55BD9ECF" Ref="#PWR09"  Part="1"
-AR Path="/55BDA313/55BD9ECF" Ref="#PWR015"  Part="1"
-AR Path="/55BDA511/55BD9ECF" Ref="#PWR027"  Part="1"
-F 0 "#PWR09" H 3475 3675 50  0001 C CNN
+AR Path="/55BDA44F/55BD9ECF" Ref="#PWR39"  Part="1"
+AR Path="/55BD9D56/55BD9ECF" Ref="#PWR27"  Part="1"
+AR Path="/55BDA313/55BD9ECF" Ref="#PWR33"  Part="1"
+AR Path="/55BDA511/55BD9ECF" Ref="#PWR45"  Part="1"
+F 0 "#PWR45" H 3475 3675 50  0001 C CNN
 F 1 "GNDA" H 3475 3775 50  0000 C CNN
 F 2 "" H 3475 3925 60  0000 C CNN
@@
 $Comp
 L LM324N-RESCUE-solarTracker U7
-U 1 1 55BD9ED5
+U 3 1 55BD9ED5
 P 4100 3225
 AR Path="/55BDA44F/55BD9ED5" Ref="U7"  Part="1"
@@
 AR Path="/55BDA511/55BD9ED5" Ref="U7"  Part="3"
 AR Path="/55BD9ED5" Ref="U4"  Part="1"
-F 0 "U4" H 4150 3425 60  0000 C CNN
+F 0 "U7" H 4150 3425 60  0000 C CNN
 F 1 "LM324N" H 4250 3025 50  0000 C CNN
 F 2 "" H 4100 3225 60  0000 C CNN
@@
 F 4 "Farnell" H 4100 3225 60  0001 C CNN "Supplier"
 F 5 "1564884" H 4100 3225 60  0001 C CNN "Order No"
-	1    4100 3225
-	1    0    0    -1
-$EndComp
-$Comp
-L +3V3 #PWR022
+	3    4100 3225
+	1    0    0    -1
+$EndComp
+$Comp
+L +3V3 #PWR40
 U 1 1 55BD9EDC
 P 4000 2625
-AR Path="/55BDA44F/55BD9EDC" Ref="#PWR022"  Part="1"
-AR Path="/55BD9D56/55BD9EDC" Ref="#PWR010"  Part="1"
-AR Path="/55BDA313/55BD9EDC" Ref="#PWR016"  Part="1"
-AR Path="/55BDA511/55BD9EDC" Ref="#PWR028"  Part="1"
-F 0 "#PWR010" H 4000 2475 50  0001 C CNN
+AR Path="/55BDA44F/55BD9EDC" Ref="#PWR40"  Part="1"
+AR Path="/55BD9D56/55BD9EDC" Ref="#PWR28"  Part="1"
+AR Path="/55BDA313/55BD9EDC" Ref="#PWR34"  Part="1"
+AR Path="/55BDA511/55BD9EDC" Ref="#PWR46"  Part="1"
+F 0 "#PWR46" H 4000 2475 50  0001 C CNN
 F 1 "+3V3" H 4000 2765 50  0000 C CNN
 F 2 "" H 4000 2625 60  0000 C CNN
@@
 AR Path="/55BDA313/55BD9EF7" Ref="R8"  Part="1"
 AR Path="/55BDA511/55BD9EF7" Ref="R18"  Part="1"
-F 0 "R3" V 5780 3225 50  0000 C CNN
+F 0 "R18" V 5780 3225 50  0000 C CNN
 F 1 "150k" V 5625 3225 50  0000 C CNN
 F 2 "" V 5630 3225 30  0000 C CNN
@@
 AR Path="/55BDA313/55BD9EFE" Ref="R9"  Part="1"
 AR Path="/55BDA511/55BD9EFE" Ref="R19"  Part="1"
-F 0 "R4" V 7430 3625 50  0000 C CNN
+F 0 "R19" V 7430 3625 50  0000 C CNN
 F 1 "33k" V 7250 3625 50  0000 C CNN
 F 2 "" V 7280 3625 30  0000 C CNN
@@
 AR Path="/55BDA313/55BD9F05" Ref="R7"  Part="1"
 AR Path="/55BDA511/55BD9F05" Ref="R17"  Part="1"
-F 0 "R2" V 5230 3225 50  0000 C CNN
+F 0 "R17" V 5230 3225 50  0000 C CNN
 F 1 "150k" V 5075 3225 50  0000 C CNN
 F 2 "" V 5080 3225 30  0000 C CNN
@@
 $EndComp
 $Comp
-L GNDA #PWR023
+L GNDA #PWR41
 U 1 1 55BD9F18
 P 5950 3975
-AR Path="/55BDA44F/55BD9F18" Ref="#PWR023"  Part="1"
-AR Path="/55BD9D56/55BD9F18" Ref="#PWR011"  Part="1"
-AR Path="/55BDA313/55BD9F18" Ref="#PWR017"  Part="1"
-AR Path="/55BDA511/55BD9F18" Ref="#PWR029"  Part="1"
-F 0 "#PWR011" H 5950 3725 50  0001 C CNN
+AR Path="/55BDA44F/55BD9F18" Ref="#PWR41"  Part="1"
+AR Path="/55BD9D56/55BD9F18" Ref="#PWR29"  Part="1"
+AR Path="/55BDA313/55BD9F18" Ref="#PWR35"  Part="1"
+AR Path="/55BDA511/55BD9F18" Ref="#PWR47"  Part="1"
+F 0 "#PWR47" H 5950 3725 50  0001 C CNN
 F 1 "GNDA" H 5950 3825 50  0000 C CNN
 F 2 "" H 5950 3975 60  0000 C CNN
@@
 AR Path="/55BDA313/55BD9F21" Ref="R10"  Part="1"
 AR Path="/55BDA511/55BD9F21" Ref="R20"  Part="1"
-F 0 "R5" V 7430 4050 50  0000 C CNN
+F 0 "R20" V 7430 4050 50  0000 C CNN
 F 1 "56k" V 7250 4050 50  0000 C CNN
 F 2 "" V 7280 4050 30  0000 C CNN
@@
 $EndComp
 $Comp
-L GNDA #PWR024
+L GNDA #PWR44
 U 1 1 55BD9F2A
 P 7350 4325
-AR Path="/55BDA44F/55BD9F2A" Ref="#PWR024"  Part="1"
-AR Path="/55BD9D56/55BD9F2A" Ref="#PWR012"  Part="1"
-AR Path="/55BDA313/55BD9F2A" Ref="#PWR018"  Part="1"
-AR Path="/55BDA511/55BD9F2A" Ref="#PWR030"  Part="1"
-F 0 "#PWR012" H 7350 4075 50  0001 C CNN
+AR Path="/55BDA44F/55BD9F2A" Ref="#PWR44"  Part="1"
+AR Path="/55BD9D56/55BD9F2A" Ref="#PWR32"  Part="1"
+AR Path="/55BDA313/55BD9F2A" Ref="#PWR38"  Part="1"
+AR Path="/55BDA511/55BD9F2A" Ref="#PWR50"  Part="1"
+F 0 "#PWR50" H 7350 4075 50  0001 C CNN
 F 1 "GNDA" H 7350 4175 50  0000 C CNN
 F 2 "" H 7350 4325 60  0000 C CNN
@@
 $EndComp
 $Comp
-L +3V3 #PWR025
+L +3V3 #PWR42
 U 1 1 55BD9F36
 P 6600 2825
-AR Path="/55BDA44F/55BD9F36" Ref="#PWR025"  Part="1"
-AR Path="/55BD9D56/55BD9F36" Ref="#PWR013"  Part="1"
-AR Path="/55BDA313/55BD9F36" Ref="#PWR019"  Part="1"
-AR Path="/55BDA511/55BD9F36" Ref="#PWR031"  Part="1"
-F 0 "#PWR013" H 6600 2675 50  0001 C CNN
+AR Path="/55BDA44F/55BD9F36" Ref="#PWR42"  Part="1"
+AR Path="/55BD9D56/55BD9F36" Ref="#PWR30"  Part="1"
+AR Path="/55BDA313/55BD9F36" Ref="#PWR36"  Part="1"
+AR Path="/55BDA511/55BD9F36" Ref="#PWR48"  Part="1"
+F 0 "#PWR48" H 6600 2675 50  0001 C CNN
 F 1 "+3V3" H 6600 2965 50  0000 C CNN
 F 2 "" H 6600 2825 60  0000 C CNN
@@
 DIO
 $Comp
-L GNDA #PWR026
+L GNDA #PWR43
 U 1 1 55BDC59E
 P 6600 4000
-AR Path="/55BDA44F/55BDC59E" Ref="#PWR026"  Part="1"
-AR Path="/55BD9D56/55BDC59E" Ref="#PWR014"  Part="1"
-AR Path="/55BDA313/55BDC59E" Ref="#PWR020"  Part="1"
-AR Path="/55BDA511/55BDC59E" Ref="#PWR032"  Part="1"
-F 0 "#PWR014" H 6600 3750 50  0001 C CNN
+AR Path="/55BDA44F/55BDC59E" Ref="#PWR43"  Part="1"
+AR Path="/55BD9D56/55BDC59E" Ref="#PWR31"  Part="1"
+AR Path="/55BDA313/55BDC59E" Ref="#PWR37"  Part="1"
+AR Path="/55BDA511/55BDC59E" Ref="#PWR49"  Part="1"
+F 0 "#PWR49" H 6600 3750 50  0001 C CNN
 F 1 "GNDA" H 6600 3850 50  0000 C CNN
 F 2 "" H 6600 4000 60  0000 C CNN
@@
 AR Path="/55BDA313/55BDDF51" Ref="C14"  Part="1"
 AR Path="/55BDA511/55BDDF51" Ref="C18"  Part="1"
-F 0 "C12" V 7125 2850 50  0000 L CNN
+F 0 "C18" V 7125 2850 50  0000 L CNN
 F 1 "470n" H 7000 2800 50  0000 L CNN
 F 2 "" H 7013 2750 30  0000 C CNN
@@
 $Comp
 L LM324N-RESCUE-solarTracker U7
-U 2 1 55BDFBFD
+U 4 1 55BDFBFD
 P 6700 3325
 AR Path="/55BDA44F/55BDFBFD" Ref="U7"  Part="2"
@@
 AR Path="/55BDA511/55BDFBFD" Ref="U7"  Part="4"
 AR Path="/55BDFBFD" Ref="U4"  Part="2"
-F 0 "U4" H 6750 3525 60  0000 C CNN
+F 0 "U7" H 6750 3525 60  0000 C CNN
 F 1 "LM324N" H 6850 3125 50  0000 C CNN
 F 2 "" H 6700 3325 60  0000 C CNN
 F 3 "" H 6700 3325 60  0000 C CNN
-	2    6700 3325
+	4    6700 3325
 	1    0    0    -1
 $EndComp
@@
 AR Path="/55BDA44F/55BD33E1" Ref="C15"  Part="1"
 AR Path="/55BDA511/55BD33E1" Ref="C17"  Part="1"
-F 0 "C11" H 6025 3750 50  0000 L CNN
+F 0 "C17" H 6025 3750 50  0000 L CNN
 F 1 "470n" H 5975 3525 50  0000 L CNN
 F 2 "" H 5988 3475 30  0000 C CNN

Commit message: footprint generation, chibiOS and chibiOS-servo libraries
Connections:
- net DIO: now also U7.7; no longer U7.14
- net at C11.2, R13.1: now also U7.5 (+); no longer U7.12 (+)
- net at U6.2 (C): now also U7.2 (-); no longer U7.9 (-)
- net at R11.1: now also U7.3 (+); no longer U7.10 (+)
- net at R11.2, R12.2: now also U7.1; no longer U7.8
- net at R14.1, R15.2: now also U7.6 (-); no longer U7.13 (-)
Changed lines of the file:
@@
 LIBS:swd
 LIBS:lm2577
+LIBS:lm2596
 LIBS:solarTracker-cache
 EELAYER 25 0
@@
 AR Path="/55BDA313/55BD9EC1" Ref="U5"  Part="1"
 AR Path="/55BDA511/55BD9EC1" Ref="U8"  Part="1"
-F 0 "U8" H 3350 3600 60  0000 C CNN
+F 0 "U3" H 3350 3600 60  0000 C CNN
 F 1 "photodiode" H 3350 3600 60  0000 C CNN
 F 2 "" H 3350 3600 60  0000 C CNN
@@
 AR Path="/55BDA313/55BD9EC8" Ref="R6"  Part="1"
 AR Path="/55BDA511/55BD9EC8" Ref="R16"  Part="1"
-F 0 "R16" V 4425 2750 50  0000 C CNN
+F 0 "R1" V 4425 2750 50  0000 C CNN
 F 1 "UNREGULATED" V 4525 2775 50  0000 C CNN
 F 2 "" V 4330 2750 30  0000 C CNN
@@
 AR Path="/55BDA313/55BD9ECF" Ref="#PWR33"  Part="1"
 AR Path="/55BDA511/55BD9ECF" Ref="#PWR45"  Part="1"
-F 0 "#PWR45" H 3475 3675 50  0001 C CNN
+F 0 "#PWR27" H 3475 3675 50  0001 C CNN
 F 1 "GNDA" H 3475 3775 50  0000 C CNN
 F 2 "" H 3475 3925 60  0000 C CNN
@@
 $Comp
 L LM324N-RESCUE-solarTracker U7
-U 3 1 55BD9ED5
+U 1 1 55BD9ED5
 P 4100 3225
 AR Path="/55BDA44F/55BD9ED5" Ref="U7"  Part="1"
@@
 AR Path="/55BDA511/55BD9ED5" Ref="U7"  Part="3"
 AR Path="/55BD9ED5" Ref="U4"  Part="1"
-F 0 "U7" H 4150 3425 60  0000 C CNN
+F 0 "U4" H 4150 3425 60  0000 C CNN
 F 1 "LM324N" H 4250 3025 50  0000 C CNN
 F 2 "" H 4100 3225 60  0000 C CNN
@@
 F 4 "Farnell" H 4100 3225 60  0001 C CNN "Supplier"
 F 5 "1564884" H 4100 3225 60  0001 C CNN "Order No"
-	3    4100 3225
+	1    4100 3225
 	1    0    0    -1
 $EndComp
@@
 AR Path="/55BDA313/55BD9EDC" Ref="#PWR34"  Part="1"
 AR Path="/55BDA511/55BD9EDC" Ref="#PWR46"  Part="1"
-F 0 "#PWR46" H 4000 2475 50  0001 C CNN
+F 0 "#PWR28" H 4000 2475 50  0001 C CNN
 F 1 "+3V3" H 4000 2765 50  0000 C CNN
 F 2 "" H 4000 2625 60  0000 C CNN
@@
 AR Path="/55BDA313/55BD9EF7" Ref="R8"  Part="1"
 AR Path="/55BDA511/55BD9EF7" Ref="R18"  Part="1"
-F 0 "R18" V 5780 3225 50  0000 C CNN
+F 0 "R3" V 5780 3225 50  0000 C CNN
 F 1 "150k" V 5625 3225 50  0000 C CNN
 F 2 "" V 5630 3225 30  0000 C CNN
@@
 AR Path="/55BDA313/55BD9EFE" Ref="R9"  Part="1"
 AR Path="/55BDA511/55BD9EFE" Ref="R19"  Part="1"
-F 0 "R19" V 7430 3625 50  0000 C CNN
+F 0 "R4" V 7430 3625 50  0000 C CNN
 F 1 "33k" V 7250 3625 50  0000 C CNN
 F 2 "" V 7280 3625 30  0000 C CNN
@@
 AR Path="/55BDA313/55BD9F05" Ref="R7"  Part="1"
 AR Path="/55BDA511/55BD9F05" Ref="R17"  Part="1"
-F 0 "R17" V 5230 3225 50  0000 C CNN
+F 0 "R2" V 5230 3225 50  0000 C CNN
 F 1 "150k" V 5075 3225 50  0000 C CNN
 F 2 "" V 5080 3225 30  0000 C CNN
@@
 AR Path="/55BDA313/55BD9F18" Ref="#PWR35"  Part="1"
 AR Path="/55BDA511/55BD9F18" Ref="#PWR47"  Part="1"
-F 0 "#PWR47" H 5950 3725 50  0001 C CNN
+F 0 "#PWR29" H 5950 3725 50  0001 C CNN
 F 1 "GNDA" H 5950 3825 50  0000 C CNN
 F 2 "" H 5950 3975 60  0000 C CNN
@@
 AR Path="/55BDA313/55BD9F21" Ref="R10"  Part="1"
 AR Path="/55BDA511/55BD9F21" Ref="R20"  Part="1"
-F 0 "R20" V 7430 4050 50  0000 C CNN
+F 0 "R5" V 7430 4050 50  0000 C CNN
 F 1 "56k" V 7250 4050 50  0000 C CNN
 F 2 "" V 7280 4050 30  0000 C CNN
@@
 AR Path="/55BDA313/55BD9F2A" Ref="#PWR38"  Part="1"
 AR Path="/55BDA511/55BD9F2A" Ref="#PWR50"  Part="1"
-F 0 "#PWR50" H 7350 4075 50  0001 C CNN
+F 0 "#PWR32" H 7350 4075 50  0001 C CNN
 F 1 "GNDA" H 7350 4175 50  0000 C CNN
 F 2 "" H 7350 4325 60  0000 C CNN
@@
 AR Path="/55BDA313/55BD9F36" Ref="#PWR36"  Part="1"
 AR Path="/55BDA511/55BD9F36" Ref="#PWR48"  Part="1"
-F 0 "#PWR48" H 6600 2675 50  0001 C CNN
+F 0 "#PWR30" H 6600 2675 50  0001 C CNN
 F 1 "+3V3" H 6600 2965 50  0000 C CNN
 F 2 "" H 6600 2825 60  0000 C CNN
@@
 AR Path="/55BDA313/55BDC59E" Ref="#PWR37"  Part="1"
 AR Path="/55BDA511/55BDC59E" Ref="#PWR49"  Part="1"
-F 0 "#PWR49" H 6600 3750 50  0001 C CNN
+F 0 "#PWR31" H 6600 3750 50  0001 C CNN
 F 1 "GNDA" H 6600 3850 50  0000 C CNN
 F 2 "" H 6600 4000 60  0000 C CNN
@@
 AR Path="/55BDA313/55BDDF51" Ref="C14"  Part="1"
 AR Path="/55BDA511/55BDDF51" Ref="C18"  Part="1"
-F 0 "C18" V 7125 2850 50  0000 L CNN
+F 0 "C12" V 7125 2850 50  0000 L CNN
 F 1 "470n" H 7000 2800 50  0000 L CNN
 F 2 "" H 7013 2750 30  0000 C CNN
@@
 $Comp
 L LM324N-RESCUE-solarTracker U7
-U 4 1 55BDFBFD
+U 2 1 55BDFBFD
 P 6700 3325
 AR Path="/55BDA44F/55BDFBFD" Ref="U7"  Part="2"
@@
 AR Path="/55BDA511/55BDFBFD" Ref="U7"  Part="4"
 AR Path="/55BDFBFD" Ref="U4"  Part="2"
-F 0 "U7" H 6750 3525 60  0000 C CNN
+F 0 "U4" H 6750 3525 60  0000 C CNN
 F 1 "LM324N" H 6850 3125 50  0000 C CNN
 F 2 "" H 6700 3325 60  0000 C CNN
 F 3 "" H 6700 3325 60  0000 C CNN
-	4    6700 3325
+	2    6700 3325
 	1    0    0    -1
 $EndComp
@@
 AR Path="/55BDA44F/55BD33E1" Ref="C15"  Part="1"
 AR Path="/55BDA511/55BD33E1" Ref="C17"  Part="1"
-F 0 "C17" H 6025 3750 50  0000 L CNN
+F 0 "C11" H 6025 3750 50  0000 L CNN
 F 1 "470n" H 5975 3525 50  0000 L CNN
 F 2 "" H 5988 3475 30  0000 C CNN
